File: PCB_B3.kicad_pcb (KiCad board)
At the start: 2 copper layers, 17.8 x 33 mm, 18 parts, among them J1 Screw_Terminal_01x02, J2 Screw_Terminal_01x02, J3 Conn_01x03_Male, J4 Conn_01x03_Male, J5 Conn_01x04_Male, K1 G3MB202PDC12, P1 Digital, P3 ADC, P4 Analog, P5 ADC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

Commit message: Update
Parts:
- moved J1 31.5 mm to (212.1, 82.5), turned to 180 degrees
- moved F1 17.8 mm to (170.2, 72.4)
- moved U3 13.5 mm to (138.4, 119.4), turned to 0 degrees
- moved PS1 6.35 mm to (212.1, 102.9)
- moved J4 5.08 mm to (162.6, 109.2), turned to 0 degrees
- moved U2 4.02 mm to (125.7, 94.0), turned to 270 degrees
- moved J2 2.54 mm to (186.7, 82.5)
Routing:
- net GND: track 0.00 -> 119.0 mm
- net /CON_FUSE_REL_1: track 0.00 -> 105.4 mm
- net +5V: track 0.00 -> 83.0 mm
- net /13(SCK): track 0.00 -> 56.1 mm
- net /CON_TB_1: track 0.00 -> 54.7 mm
- net /4: track 0.00 -> 45.8 mm
- net /12(MISO): track 0.00 -> 43.3 mm
- net Net-(F3-Pad1): track 0.00 -> 35.1 mm
- net VCC: track 0.00 -> 33.8 mm
- net /3(**): track 0.00 -> 31.0 mm
- net /11(**/MOSI): track 0.00 -> 29.5 mm
- net Net-(F1-Pad2): track 0.00 -> 25.9 mm
- net /10(**/SS): track 0.00 -> 20.8 mm
- net /RELAY_4: track 0.00 -> 20.6 mm
- net Net-(F1-Pad1): track 0.00 -> 16.5 mm
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Other:
- board outline removed

Commit message: Update
Parts:
- moved F3 41.9 mm to (194.3, 67.3)
- moved F2 24.2 mm to (162.6, 73.7)
- moved F1 11.5 mm to (181.6, 73.7)
- moved K1 10.2 mm to (133.3, 73.7)
- moved J2 7.62 mm to (194.3, 82.5)
- moved RV1 6.48 mm to (221.0, 97.8)
Routing:
- net /CON_FUSE_REL_1: track 105.4 -> 26.5 mm
- net /RELAY_2: track 13.7 -> 46.4 mm
- net /CON_TB_1: track 54.7 -> 24.3 mm
- net Net-(F3-Pad1): track 35.1 -> 15.2 mm
- net Net-(F1-Pad1): track 16.5 -> 3.81 mm
- net +5V: track 83.0 -> 72.9 mm
- net Net-(F1-Pad2): track 25.9 -> 18.5 mm
- net /RELAY_4: track 20.6 -> 16.5 mm
Other:
- board text added: "Juan Manuel Muñoz"

Commit message: Update
Routing:
- net /CON_FUSE_REL_1: track 26.5 -> 89.1 mm
- added copper zone on B.Cu, net GND
- removed copper zone on B.Cu, net (none)
Other:
- board outline added: 105.4 x 71.1 mm

Commit message: Update
Parts:
- R1: moved to B.Cu
- moved J1 16.5 mm to (212.1, 99.1)
- moved J2 16.5 mm to (194.3, 99.1)
- moved PS1 16.5 mm to (212.1, 119.4)
- moved K1 15.3 mm to (147.3, 80.0)
- moved F1 15.3 mm to (191.8, 85.1)
- moved F2 15.3 mm to (172.7, 85.1)
- moved RV1 15.2 mm to (221.0, 113.0)
- moved F3 13.0 mm to (196.8, 80.0)
- moved R1 10.2 mm to (133.3, 101.3)
- moved U2 7.62 mm to (133.3, 94.0)
Connections:
- J4 pad 1: +3V3 -> VCC
- J5 pad 1: +3V3 -> VCC
Routing:
- net GND: track 119.0 -> 0.43 mm
- net VCC: track 33.8 -> 57.7 mm
- net /CON_TB_1: track 24.2 -> 38.5 mm
- net /RELAY_2: track 46.4 -> 32.4 mm
- net /CON_FUSE_REL_1: track 89.1 -> 76.7 mm
- net +5V: track 72.9 -> 62.1 mm
- net /5(**): track 15.2 -> 5.08 mm
- net Net-(F3-Pad1): track 15.2 -> 20.1 mm
- net Net-(F1-Pad2): track 18.5 -> 14.1 mm
- net +3V3: track 3.81 -> 0.00 mm
- net /RELAY_4: track 16.5 -> 12.8 mm
- net Net-(R1-Pad1): track 8.67 -> 7.06 mm
- removed copper zone on B.Cu, net GND
Other:
- board outline removed

Commit message: Update
Routing:
- added copper zone on B.Cu, net GND
Other:
- board outline added: 95.2 x 58.4 mm
